File: Hardware/Danyboard_M0.brd (EAGLE design)
At the start: 26.6 x 63.3 mm, 48 parts, among them J2 USD-SOCKET, J4 S2B-PH-SM4-TB, J6 CORTEX_DEBUGSMD, M1 ESP-WROOM-02, U1 ATSAMD21G-A, U2 MCP73831, U3 AP2112K-3.3V, Y1 32.768kHz

Commit message: v3.2
Parts:
- removed U$1: (no value), GClib:DANYBOARD_M0_FONTPRINT_BOTTOM
- added U$2: (no value), GClib:DANYBOARD_M0_FONTPRINT_BOTTOM_NEW
- C1, C10, C2, C3, C4, C5, C6, C7, C8, C9: device SparkFun-Capacitors:0603-CAP -> Danyboard:0603-CAP_NOSILK
- D5, D6: value MBR120 -> MBR120LSFT3G; device SparkFun-DiscreteSemi:SOD-123 -> Danyboard:SOD-123_NOSILK
- J1: value (none) -> MX-47346-0001; device SparkFun-Connectors:USB-AB-MICRO-SMD_V03 -> Danyboard:USB-AB-MICRO-SMD_V03
- J2: value USD-SOCKET -> MCSP-Q-08-A-SG; device GClib:MCSP-Q-08-A-SG-T -> Danyboard:MCSP-Q-08-A-SG-T_NOSILK
- J4: device SparkFun-Connectors:JST-2-SMD -> Danyboard:JST-2-SMD_NOSILK
- J6: value CORTEX_DEBUGSMD -> DS1031-08-2*5P8BS-4-1; device SparkFun-Connectors:SAMTECH_FTSH-105-01 -> Danyboard:SAMTECH_FTSH-105-01_NOSILK
- L1: value FB - 30Ohm -> BLM18PG300SN1D; device SparkFun-Passives:0603 -> Danyboard:0603_NOSILK
- M1: device esp-wroom-02:ESP-WROOM-02 -> Danyboard:ESP-WROOM-02_NOSILK
- R1, R10, R11, R12, R2, R3, R4, R7, R8: device SparkFun-Passives:0603-RES -> Danyboard:0603-RES_NOSILK
- R13, R14: value 1M -> 3M; device SparkFun-Passives:0603-RES -> Danyboard:0603-RES_NOSILK
- R5, R6, R9: device SparkFun-Resistors:0603-RES -> Danyboard:0603-RES_NOSILK
- S1: value RESET -> TACTB-64K-F; device SparkFun-Electromechanical:TACTILE-SWITCH-SMD -> Danyboard:TACTILE-SWITCH-SMD_NOSILK
- U1: value ATSAMD21G-A -> ATSAMD21G18A-AU; device samd21-temp:TQFP-48 -> Danyboard:TQFP-48_NOSILK
- U3: value AP2112K-3.3V -> AP2112K-3.3TRG1
- Y1: value 32.768kHz -> LFXTAL009678; device SparkFun-FreqCtrl:CRYSTAL-SMD-3.2X1.5MM -> Danyboard:CRYSTAL-SMD-3.2X1.5MM_NOSILK
Routing:
- net V_BATT: track 49.6 -> 50.1 mm
- added copper zone on layer 1, net A0
- added copper zone on layer 16, net D2
- added copper zone on layer 1, net N$10
- added copper zone on layer 1, net N$13
- added copper zone on layer 16, net N$16
