File: Hardware/Danyboard_M0.sch (EAGLE design)
At the start: 47 parts, among them J2 USD-SOCKET, J4 S2B-PH-SM4-TB, J6 CORTEX_DEBUGSMD, M1 ESP-WROOM-02, U1 ATSAMD21G-A, U2 MCP73831, U3 AP2112K-3.3V, Y1 32.768kHz

Commit message: v3.2
Parts:
- C1, C10, C2, C3, C4, C5, C6, C7, C8, C9: device SparkFun-Capacitors:CAP0603-CAP -> Danyboard:CAP0603-CAP_NS
- D5, D6: value MBR120 -> MBR120LSFT3G; device SparkFun-DiscreteSemi:DIODESOD123 -> Danyboard:DIODESOD123_NS
- J1: value (none) -> MX-47346-0001; device SparkFun-Connectors:USB-ABCONN-11794 -> Danyboard:USB-ABCONN-11794
- J2: value USD-SOCKET -> MCSP-Q-08-A-SG; device GClib:USD-SOCKET -> Danyboard:USD-SOCKET-NS
- J4: device SparkFun-Connectors:M02-JST-2MM-SMT -> Danyboard:M02-JST-2MM-SMT_NS
- J6: value CORTEX_DEBUGSMD -> DS1031-08-2*5P8BS-4-1; device SparkFun-Connectors:CORTEX_DEBUGSMD -> Danyboard:CORTEX_DEBUGSMD2
- L1: value FB - 30Ohm -> BLM18PG300SN1D; device SparkFun-Passives:INDUCTOR0603 -> Danyboard:INDUCTOR0603_NS
- M1: device esp-wroom-02:ESP-WROOM-02FRONT-FACE -> Danyboard:ESP-WROOM-02-NS
- R1, R10, R11, R12, R2, R3, R4, R7, R8: device SparkFun-Passives:RESISTOR0603-RES -> Danyboard:RESISTOR0603-NS
- R13, R14: value 1M -> 3M; device SparkFun-Passives:RESISTOR0603-RES -> Danyboard:RESISTOR0603-NS
- R5, R6, R9: device SparkFun-Resistors:330OHM1/10W1%(0603) -> Danyboard:RESISTOR0603-NS
- S1: value RESET -> TACTB-64K-F; device SparkFun-Electromechanical:SWITCH-MOMENTARY-2SMD -> Danyboard:SWITCH-MOMENTARY-2SMD-NS
- U1: value ATSAMD21G-A -> ATSAMD21G18A-AU; device samd21-temp:ATSAMD21G-A -> Danyboard:ATSAMD21G-A2
- U3: value AP2112K-3.3V -> AP2112K-3.3TRG1
- Y1: value 32.768kHz -> LFXTAL009678; device SparkFun-FreqCtrl:CRYSTAL3.2X1.5MM -> Danyboard:CRYSTAL3.2X1.5MM_NS
